Commit message: add wild mujoco

File: wild/robot.urdf (robot description, URDF)
Before this commit: robot wild, 1 links, 0 joints
Links:
- added link ankle, mass 0.0230191; collision mesh filename=package://assets/servo_bracket_btm.stl; collision mesh filename=package://assets/servo_bracket_top.stl
- added link ankle_2, mass 0.0230191; collision mesh filename=package://assets/servo_bracket_btm.stl; collision mesh filename=package://assets/servo_bracket_top.stl
- added link chassis, mass 0.841214; collision mesh filename=package://assets/battery_hook.stl; collision mesh filename=package://assets/battery_hook.stl
- added link left_foot, mass 0.413618; collision mesh filename=package://assets/btm_btm_back.stl; collision mesh filename=package://assets/btm_btm_front.stl
- added link left_hip, mass 0.0849728; collision mesh filename=package://assets/hip_gear.stl; collision mesh filename=package://assets/hip_servo_gear.stl
- added link lower_leg, mass 0.380663; collision mesh filename=package://assets/htd_45h_1circle.stl; collision mesh filename=package://assets/knee_ball_low_leg_connect.stl
- added link lower_leg_2, mass 0.380663; collision mesh filename=package://assets/htd_45h_1circle.stl; collision mesh filename=package://assets/knee_ball_low_leg_connect.stl
- added link right_foot, mass 0.413618; collision mesh filename=package://assets/btm_btm_back.stl; collision mesh filename=package://assets/btm_btm_front.stl
- added link right_hip, mass 0.0849728; collision mesh filename=package://assets/hip_gear.stl; collision mesh filename=package://assets/hip_servo_gear.stl
- added link upper_leg, mass 0.236189; collision mesh filename=package://assets/htd_45h_1circle.stl; collision mesh filename=package://assets/knee_ball_left.stl
- added link upper_leg_2, mass 0.236189; collision mesh filename=package://assets/htd_45h_1circle.stl; collision mesh filename=package://assets/knee_ball_left.stl
- link waist: mass 1e-09 -> 0.438621
Joints:
- added joint left_ankle: type revolute, parent lower_leg, child ankle, origin xyz=-4.74705e-05 -0.179984 0.000442075 rpy=0.00142308 0.000132648 0.523599, axis 0 0 1, limit lower=0 upper=0 effort=10 velocity=10
- added joint left_foot: type revolute, parent ankle, child left_foot, origin xyz=-0.0268 -0.0594 0.0268 rpy=1.5708 -0.349066 1.5708, axis 0 0 1, limit lower=0 upper=0 effort=10 velocity=10
- added joint left_hip: type revolute, parent left_hip, child upper_leg, origin xyz=-0.0268591 -0.00149279 -0.0365475 rpy=8.076e-13 1.56997 0.0505006, axis 0 0 1, limit lower=-0.889656 upper=0.506607 effort=10 velocity=10
- added joint left_knee: type revolute, parent upper_leg, child lower_leg, origin xyz=0.00366073 0.194183 0.0267 rpy=-0.573319 -1.57079 -2.72581, axis 0 0 1, limit lower=-2.92267e-10 upper=1.5708 effort=10 velocity=10
- added joint left_waist_hip: type revolute, parent waist, child left_hip, origin xyz=0.0535826 -0.000150648 -0.0532864 rpy=-1.57196 9.6369e-07 1.57162, axis 0 0 1, limit lower=-0.572933 upper=1.52146 effort=10 velocity=10
- added joint right_ankle: type revolute, parent lower_leg_2, child ankle_2, origin xyz=-4.74705e-05 0.179984 0.049 rpy=-3.14017 -0.000132648 -0.523599, axis 0 0 1, limit lower=-1.0472 upper=1.11022e-16 effort=10 velocity=10
- added joint right_foot: type revolute, parent ankle_2, child right_foot, origin xyz=-0.0268 -0.0594 0.0268 rpy=1.5708 -0.349066 -1.5708, axis 0 0 1, limit lower=0 upper=0 effort=10 velocity=10
- added joint right_hip: type revolute, parent right_hip, child upper_leg_2, origin xyz=0.0266221 -0.00204462 -0.0364525 rpy=-3.14159 -1.56997 3.07001, axis 0 0 1, limit lower=-0.343431 upper=1.05283 effort=10 velocity=10
- added joint right_knee: type revolute, parent upper_leg_2, child lower_leg_2, origin xyz=0.022434 0.192305 0.0266985 rpy=3.05759 -1.56996 -3.06206, axis 0 0 1, limit lower=-1.57073 upper=6.60353e-05 effort=10 velocity=10
- added joint right_waist_hip: type revolute, parent waist, child right_hip, origin xyz=-0.0536174 -0.000245589 -0.0532864 rpy=-1.57196 9.6369e-07 -1.56997, axis 0 0 1, limit lower=-1.50038 upper=0.594017 effort=10 velocity=10
- added joint waist: type revolute, parent waist, child chassis, origin xyz=2.43399e-05 -0.000217894 0.0284972 rpy=3.14043 0.000826419 -9.6369e-07, axis 0 0 1, limit lower=-1.5708 upper=1.5708 effort=10 velocity=10
